Commit message: 已经装配好雷达，编写好启动luanch文件

File: my_robot_description/urdf/xacro/gazebo/my_robot_base_gazebo.xacro (robot description, xacro)
@@ -1,176 +1,225 @@
 <?xml version="1.0"?>
 <robot name="my_robot" xmlns:xacro="http://www.ros.org/wiki/xacro">
-    <!-- PROPERTY LIST -->
-    <xacro:property name="M_PI" value="3.1415926"/>
-    <xacro:property name="base_mass"   value="20" />
+    <xacro:property name="base_mass" value="0.1"/>
     <xacro:property name="base_radius" value="0.20"/>
     <xacro:property name="base_length" value="0.16"/>
-    <xacro:property name="wheel_mass"   value="2" />
-    <xacro:property name="wheel_radius" value="0.06"/>
-    <xacro:property name="wheel_length" value="0.025"/>
+    <xacro:property name="wheel_mass" value="0.1"/>
+    <xacro:property name="wheel_radius" value="0.025"/>
+    <xacro:property name="wheel_length" value="0.02"/>
     <xacro:property name="wheel_joint_y" value="0.19"/>
-    <xacro:property name="wheel_joint_z" value="0.05"/>
-    <xacro:property name="caster_mass"    value="0.5" />
-    <xacro:property name="caster_radius"  value="0.015"/> <!-- wheel_radius - ( base_length/2 - wheel_joint_z) -->
-    <xacro:property name="caster_joint_x" value="0.18"/>
-    <!-- Defining the colors used in this robot -->
-    <material name="yellow">
-        <color rgba="1 0.4 0 1"/>
-    </material>
-    <material name="black">
-        <color rgba="0 0 0 0.95"/>
-    </material>
-    <material name="gray">
-        <color rgba="0.75 0.75 0.75 1"/>
-    </material>
-    <!-- Macro for inertia matrix -->
-    <xacro:macro name="sphere_inertial_matrix" params="m r">
-        <inertial>
-            <mass value="${m}" />
-            <inertia ixx="${2*m*r*r/5}" ixy="0" ixz="0"
-                iyy="${2*m*r*r/5}" iyz="0"
-                izz="${2*m*r*r/5}" />
-        </inertial>
-    </xacro:macro>
-    <xacro:macro name="cylinder_inertial_matrix" params="m r h">
-        <inertial>
-            <mass value="${m}" />
-            <inertia ixx="${m*(3*r*r+h*h)/12}" ixy = "0" ixz = "0"
-                iyy="${m*(3*r*r+h*h)/12}" iyz = "0"
-                izz="${m*r*r/2}" />
-        </inertial>
-    </xacro:macro>
-    <!-- Macro for robot wheel -->
-    <xacro:macro name="wheel" params="prefix reflect">
-        <joint name="${prefix}_wheel_joint" type="continuous">
-            <origin xyz="0 ${reflect*wheel_joint_y} ${-wheel_joint_z}" rpy="0 0 0"/>
-            <parent link="base_link"/>
-            <child link="${prefix}_wheel_link"/>
-            <axis xyz="0 1 0"/>
-        </joint>
-        <link name="${prefix}_wheel_link">
-            <visual>
-                <origin xyz="0 0 0" rpy="${M_PI/2} 0 0" />
-                <geometry>
-                    <cylinder radius="${wheel_radius}" length = "${wheel_length}"/>
-                </geometry>
-                <material name="gray" />
-            </visual>
-            <collision>
-                <origin xyz="0 0 0" rpy="${M_PI/2} 0 0" />
-                <geometry>
-                    <cylinder radius="${wheel_radius}" length = "${wheel_length}"/>
-                </geometry>
-            </collision>
-            <xacro:cylinder_inertial_matrix  m="${wheel_mass}" r="${wheel_radius}" h="${wheel_length}" />
-        </link>
-        <gazebo reference="${prefix}_wheel_link">
-            <material>Gazebo/Gray</material>
-        </gazebo>
-        <!-- Transmission is important to link the joints and the controller -->
-        <transmission name="${prefix}_wheel_joint_trans">
-            <type>transmission_interface/SimpleTransmission</type>
-            <joint name="${prefix}_wheel_joint" >
-                <hardwareInterface>hardware_interface/VelocityJointInterface</hardwareInterface>
-            </joint>
-            <actuator name="${prefix}_wheel_joint_motor">
-                <hardwareInterface>hardware_interface/VelocityJointInterface</hardwareInterface>
-                <mechanicalReduction>1</mechanicalReduction>
-            </actuator>
-        </transmission>
-    </xacro:macro>
-    <!-- Macro for robot caster -->
-    <xacro:macro name="caster" params="prefix reflect">
-        <joint name="${prefix}_caster_joint" type="continuous">
-            <origin xyz="${reflect*caster_joint_x} 0 ${-(base_length/2 + caster_radius)}" rpy="0 0 0"/>
-            <parent link="base_link"/>
-            <child link="${prefix}_caster_link"/>
-            <axis xyz="0 1 0"/>
-        </joint>
-        <link name="${prefix}_caster_link">
-            <visual>
-                <origin xyz="0 0 0" rpy="0 0 0"/>
-                <geometry>
-                    <sphere radius="${caster_radius}" />
-                </geometry>
-                <material name="black" />
-            </visual>
-            <collision>
-                <origin xyz="0 0 0" rpy="0 0 0"/>
-                <geometry>
-                    <sphere radius="${caster_radius}" />
-                </geometry>
-            </collision>
-            <sphere_inertial_matrix  m="${caster_mass}" r="${caster_radius}" />
-        </link>
-        <gazebo reference="${prefix}_caster_link">
-            <material>Gazebo/Black</material>
-        </gazebo>
-    </xacro:macro>
-    <xacro:macro name="my_robot_base_gazebo">
-        <link name="base_footprint">
-            <visual>
-                <origin xyz="0 0 0" rpy="0 0 0" />
-                <geometry>
-                    <box size="0.001 0.001 0.001" />
-                </geometry>
-            </visual>
-        </link>
-        <gazebo reference="base_footprint">
-            <turnGravityOff>false</turnGravityOff>
-        </gazebo>
-        <joint name="base_footprint_joint" type="fixed">
-            <origin xyz="0 0 ${base_length/2 + caster_radius*2}" rpy="0 0 0" />
-            <parent link="base_footprint"/>
-            <child link="base_link" />
-        </joint>
-        <link name="base_link">
-            <visual>
-                <origin xyz=" 0 0 0" rpy="0 0 0" />
-                <geometry>
-                    <cylinder length="${base_length}" radius="${base_radius}"/>
-                </geometry>
-                <material name="yellow" />
-            </visual>
-            <collision>
-                <origin xyz=" 0 0 0" rpy="0 0 0" />
-                <geometry>
-                    <cylinder length="${base_length}" radius="${base_radius}"/>
-                </geometry>
-            </collision>
-            <xacro:cylinder_inertial_matrix  m="${base_mass}" r="${base_radius}" h="${base_length}" />
-        </link>
-        <gazebo reference="base_link">
-            <material>Gazebo/Blue</material>
-        </gazebo>
-        <wheel prefix="left"  reflect="-1"/>
-        <wheel prefix="right" reflect="1"/>
-        <caster prefix="front" reflect="-1"/>
-        <caster prefix="back"  reflect="1"/>
-        <!-- controller -->
-        <gazebo>
-            <plugin name="differential_drive_controller"
-                    filename="libgazebo_ros_diff_drive.so">
-                <rosDebugLevel>Debug</rosDebugLevel>
-                <publishWheelTF>true</publishWheelTF>
-                <robotNamespace>/</robotNamespace>
-                <publishTf>1</publishTf>
-                <publishWheelJointState>true</publishWheelJointState>
-                <alwaysOn>true</alwaysOn>
-                <updateRate>100.0</updateRate>
-                <legacyMode>true</legacyMode>
-                <leftJoint>left_wheel_joint</leftJoint>
-                <rightJoint>right_wheel_joint</rightJoint>
-                <wheelSeparation>${wheel_joint_y*2}</wheelSeparation>
-                <wheelDiameter>${2*wheel_radius}</wheelDiameter>
-                <broadcastTF>1</broadcastTF>
-                <wheelTorque>30</wheelTorque>
-                <wheelAcceleration>1.8</wheelAcceleration>
-                <commandTopic>cmd_vel</commandTopic>
-                <odometryFrame>odom</odometryFrame>
-                <odometryTopic>odom</odometryTopic>
-                <robotBaseFrame>base_footprint</robotBaseFrame>
-            </plugin>
-        </gazebo>
-    </xacro:macro>
+    <xacro:property name="caster_radius" value="0.025"/>
+    <link name="base_footprint"/>
+    <joint name="base_joint" type="fixed">
+        <parent link="base_footprint"/>
+        <child link="base_link"/>
+        <origin rpy="0 0 0 " xyz="7 4 0.025"/>
+    </joint>
+    <link name="base_link">
+        <visual>
+            <geometry>
+                <box size="0.25 0.16 0.05"/>
+            </geometry>
+            <origin rpy="0 0 0 " xyz="0 0 0 "/>
+            <!-- <material name="blue">
+                <color rgba="0 0 0.8 1"/>
+            </material> -->
+        </visual>
+        <collision>
+            <origin rpy="0 0 0 " xyz="0 0 0 "/>
+            <geometry>
+                <box size="0.25 0.16 0.05"/>
+            </geometry>
+        </collision>
+        <inertial>
+            <origin rpy="0 0 0 " xyz="0 0 0 "/>
+            <mass value="${base_mass}"/>
+            <inertia
+                ixx="0.0001"
+                iyy="0.0001"
+                ixy="0"
+                ixz="0"
+                iyz="0"
+                izz="0.0001"/>
+        </inertial>
+    </link>
+    <joint name="left_wheel_joint1" type="continuous">
+        <origin xyz="0.1 0.09 -0.03" rpy="1.5707 0 0"/>
+        <parent link="base_link"/>
+        <child link="left_wheel_link1"/>
+        <axis xyz="0 0 -1"/>
+    </joint>
+    <link name="left_wheel_link1">
+        <visual>
+            <geometry>
+                <cylinder radius="${wheel_radius}" length="${wheel_length}"/>
+            </geometry>
+            <material name="black">
+                <color rgba="0 0 0 1"/>
+            </material>
+        </visual>
+        <collision>
+            <origin xyz="0 0 0" rpy="0 0 0 "/>
+            <geometry>
+                <cylinder radius="${wheel_radius}" length="${wheel_length}"/>
+            </geometry>
+        </collision>
+        <inertial>
+           <mass value="${wheel_mass}"/>
+            <inertia
+                ixx="0.0001"
+                iyy="0.0001"
+                ixy="0"
+                ixz="0"
+                iyz="0"
+                izz="0.0001"/>
+            <origin xyz="0 0 0" rpy="0 0 0 "/>
+        </inertial>
+    </link>
+    <joint name="right_wheel_joint1" type="continuous">
+        <origin xyz="0.1 -0.09 -0.03" rpy="1.5707 0 0"/>
+        <parent link="base_link"/>
+        <child link="right_wheel_link1"/>
+        <axis xyz="0 0 -1"/>
+    </joint>
+    <link name="right_wheel_link1">
+        <visual>
+            <geometry>
+                <cylinder radius="${wheel_radius}" length="${wheel_length}"/>
+            </geometry>
+            <material name="black">
+                <color rgba="0 0 0 1"/>
+            </material>
+        </visual>
+        <collision>
+            <origin xyz="0 0 0" rpy="0 0 0 "/>
+            <geometry>
+                <cylinder radius="${wheel_radius}" length="${wheel_length}"/>
+            </geometry>
+        </collision>
+        <inertial>
+            <mass value="${wheel_mass}"/>
+            <inertia
+                ixx="0.0001"
+                iyy="0.0001"
+                ixy="0"
+                ixz="0"
+                iyz="0"
+                izz="0.0001"/>
+            <origin xyz="0 0 0" rpy="0 0 0 "/>
+        </inertial>
+    </link>
+    <joint name="left_wheel_joint2" type="continuous">
+    <origin xyz="-0.1 0.09 -0.03" rpy="1.5707 0 0"/>
+    <parent link="base_link"/>
+    <child link="left_wheel_link2"/>
+    <axis xyz="0 0 -1"/>
+</joint>
+<link name="left_wheel_link2">
+    <visual>
+        <geometry>
+            <cylinder radius="${wheel_radius}" length="${wheel_length}"/>
+        </geometry>
+        <material name="black">
+            <color rgba="0 0 0 1"/>
+        </material>
+    </visual>
+    <collision>
+        <origin xyz="0 0 0" rpy="0 0 0 "/>
+        <geometry>
+            <cylinder radius="${wheel_radius}" length="${wheel_length}"/>
+        </geometry>
+    </collision>
+    <inertial>
+        <mass value="${wheel_mass}"/>
+        <inertia
+            ixx="0.0001"
+            iyy="0.0001"
+            ixy="0"
+            ixz="0"
+            iyz="0"
+            izz="0.0001"/>
+        <origin xyz="0 0 0" rpy="0 0 0 "/>
+    </inertial>
+</link>
+<joint name="right_wheel_joint2" type="continuous">
+    <origin xyz="-0.1 -0.09 -0.03" rpy="1.5707 0 0"/>
+    <parent link="base_link"/>
+    <child link="right_wheel_link2"/>
+    <axis xyz="0 0 -1"/>
+</joint>
+<link name="right_wheel_link2">
+    <visual>
+        <geometry>
+            <cylinder radius="${wheel_radius}" length="${wheel_length}"/>
+        </geometry>
+        <material name="black">
+            <color rgba="0 0 0 1"/>
+        </material>
+    </visual>
+    <collision>
+        <origin xyz="0 0 0" rpy="0 0 0 "/>
+        <geometry>
+            <cylinder radius="${wheel_radius}" length="${wheel_length}"/>
+        </geometry>
+    </collision>
+    <inertial>
+        <mass value="${wheel_mass}"/>
+        <inertia
+            ixx="0.0001"
+            iyy="0.0001"
+            ixy="0"
+            ixz="0"
+            iyz="0"
+            izz="0.0001"/>
+        <origin xyz="0 0 0" rpy="0 0 0 "/>
+    </inertial>
+</link>
+<link name="laser_link">
+    <visual>
+        <geometry>
+            <cylinder length="0.06" radius="0.04"/>
+        </geometry>
+        <material name="white">
+            <color rgba="1 1 1 1"/>
+        </material>
+    </visual>
+</link>
+<joint name="laser_joint" type="fixed">
+    <parent link="base_link"/>
+    <child link="laser_link"/>
+    <origin xyz="0 0.0 0.06"/>
+</joint>
+    <!-- <joint name="caster_joint" type="continuous">
+        <origin xyz="0 0 0" rpy="-0.10 0 -0.03"/>
+        <parent link="base_link"/>
+        <child link="caster_link"/>
+        <axis xyz="0 0 1"/>
+    </joint>
+    <link name="caster_link">
+        <visual>
+            <geometry>
+                <sphere radius="${caster_radius}"/>
+            </geometry>
+            <material name="black">
+                <color rgba="0 0 0 1"/>
+            </material>
+        </visual>
+        <collision>
+            <origin xyz="0 0 0" rpy="0 0 0"/>
+            <geometry>
+                <sphere radius="${caster_radius}"/>
+            </geometry>
+        </collision>
+        <inertial>
+            <mass value="${wheel_mass}"/>
+            <origin xyz="0 0 0" rpy="0 0 0"/>
+            <inertia
+                ixx="0"
+                iyy="0"
+                ixy="0"
+                ixz="0"
+                iyz="0"
+                izz="0"/>
+        </inertial>
+    </link> -->
 </robot>
