Commit message: 暂存一下

File: my_robot_description/urdf/xacro/gazebo/my_robot_base_gazebo.xacro (robot description, xacro)
@@ -1,4 +1,6 @@
 <?xml version="1.0"?>
 <robot name="my_robot" xmlns:xacro="http://www.ros.org/wiki/xacro">
+    <xacro:include filename="$(find my_robot_description)/urdf/xacro/gazebo/my_robot_control.xacro" />
+    <xacro:include filename="$(find my_robot_description)/urdf/xacro/gazebo/my_robot_with_laser_gazebo.xacro" />
     <xacro:property name="base_mass" value="0.1"/>
     <xacro:property name="base_radius" value="0.20"/>
@@ -9,5 +11,35 @@
     <xacro:property name="wheel_joint_y" value="0.19"/>
     <xacro:property name="caster_radius" value="0.025"/>
-    <link name="base_footprint"/>
+    <link name="base_footprint">
+        <origin rpy="0 0 0 " xyz="0 0 0"/>
+    </link>
+    <link name="base_link">
+        <visual>
+            <geometry>
+                <box size="0.25 0.16 0.05"/>
+            </geometry>
+            <origin rpy="0 0 0 " xyz="0 0 0 "/>
+            <!-- <material name="blue">
+                <color rgba="0 0 0.8 1"/>
+            </material> -->
+        </visual>
+        <collision>
+            <origin rpy="0 0 0 " xyz="0 0 0 "/>
+            <geometry>
+                <box size="0.25 0.16 0.05"/>
+            </geometry>
+        </collision>
+        <inertial>
+            <origin rpy="0 0 0 " xyz="0 0 0 "/>
+            <mass value="${base_mass}"/>
+            <inertia
+                ixx="0.0001"
+                iyy="0.0001"
+                ixy="0"
+                ixz="0"
+                iyz="0"
+                izz="0.0001"/>
+        </inertial>
+    </link>
     <joint name="base_joint" type="fixed">
         <parent link="base_footprint"/>
@@ -15,30 +47,29 @@
         <origin rpy="0 0 0 " xyz="7 4 0.025"/>
     </joint>
-    <link name="base_link">
-        <visual>
-            <geometry>
-                <box size="0.25 0.16 0.05"/>
-            </geometry>
-            <origin rpy="0 0 0 " xyz="0 0 0 "/>
-            <!-- <material name="blue">
-                <color rgba="0 0 0.8 1"/>
-            </material> -->
-        </visual>
-        <collision>
-            <origin rpy="0 0 0 " xyz="0 0 0 "/>
-            <geometry>
-                <box size="0.25 0.16 0.05"/>
-            </geometry>
-        </collision>
-        <inertial>
-            <origin rpy="0 0 0 " xyz="0 0 0 "/>
-            <mass value="${base_mass}"/>
-            <inertia
-                ixx="0.0001"
-                iyy="0.0001"
-                ixy="0"
-                ixz="0"
-                iyz="0"
-                izz="0.0001"/>
+    <link name="left_wheel_link1">
+        <visual>
+            <geometry>
+                <cylinder radius="${wheel_radius}" length="${wheel_length}"/>
+            </geometry>
+            <material name="black">
+                <color rgba="0 0 0 1"/>
+            </material>
+        </visual>
+        <collision>
+            <origin xyz="0 0 0" rpy="0 0 0 "/>
+            <geometry>
+                <cylinder radius="${wheel_radius}" length="${wheel_length}"/>
+            </geometry>
+        </collision>
+        <inertial>
+           <mass value="${wheel_mass}"/>
+            <inertia
+                ixx="0.0001"
+                iyy="0.0001"
+                ixy="0"
+                ixz="0"
+                iyz="0"
+                izz="0.0001"/>
+            <origin xyz="0 0 0" rpy="0 0 0 "/>
         </inertial>
     </link>
@@ -49,21 +80,21 @@
         <axis xyz="0 0 -1"/>
     </joint>
-    <link name="left_wheel_link1">
-        <visual>
-            <geometry>
-                <cylinder radius="${wheel_radius}" length="${wheel_length}"/>
-            </geometry>
-            <material name="black">
-                <color rgba="0 0 0 1"/>
-            </material>
-        </visual>
-        <collision>
-            <origin xyz="0 0 0" rpy="0 0 0 "/>
-            <geometry>
-                <cylinder radius="${wheel_radius}" length="${wheel_length}"/>
-            </geometry>
-        </collision>
-        <inertial>
-           <mass value="${wheel_mass}"/>
+    <link name="right_wheel_link1">
+        <visual>
+            <geometry>
+                <cylinder radius="${wheel_radius}" length="${wheel_length}"/>
+            </geometry>
+            <material name="black">
+                <color rgba="0 0 0 1"/>
+            </material>
+        </visual>
+        <collision>
+            <origin xyz="0 0 0" rpy="0 0 0 "/>
+            <geometry>
+                <cylinder radius="${wheel_radius}" length="${wheel_length}"/>
+            </geometry>
+        </collision>
+        <inertial>
+            <mass value="${wheel_mass}"/>
             <inertia
                 ixx="0.0001"
@@ -82,5 +113,5 @@
         <axis xyz="0 0 -1"/>
     </joint>
-    <link name="right_wheel_link1">
+    <link name="left_wheel_link2">
         <visual>
             <geometry>
@@ -110,84 +141,57 @@
     </link>
     <joint name="left_wheel_joint2" type="continuous">
-    <origin xyz="-0.1 0.09 -0.03" rpy="1.5707 0 0"/>
-    <parent link="base_link"/>
-    <child link="left_wheel_link2"/>
-    <axis xyz="0 0 -1"/>
-</joint>
-<link name="left_wheel_link2">
-    <visual>
-        <geometry>
-            <cylinder radius="${wheel_radius}" length="${wheel_length}"/>
-        </geometry>
-        <material name="black">
-            <color rgba="0 0 0 1"/>
-        </material>
-    </visual>
-    <collision>
-        <origin xyz="0 0 0" rpy="0 0 0 "/>
-        <geometry>
-            <cylinder radius="${wheel_radius}" length="${wheel_length}"/>
-        </geometry>
-    </collision>
-    <inertial>
-        <mass value="${wheel_mass}"/>
-        <inertia
-            ixx="0.0001"
-            iyy="0.0001"
-            ixy="0"
-            ixz="0"
-            iyz="0"
-            izz="0.0001"/>
-        <origin xyz="0 0 0" rpy="0 0 0 "/>
-    </inertial>
-</link>
-<joint name="right_wheel_joint2" type="continuous">
-    <origin xyz="-0.1 -0.09 -0.03" rpy="1.5707 0 0"/>
-    <parent link="base_link"/>
-    <child link="right_wheel_link2"/>
-    <axis xyz="0 0 -1"/>
-</joint>
-<link name="right_wheel_link2">
-    <visual>
-        <geometry>
-            <cylinder radius="${wheel_radius}" length="${wheel_length}"/>
-        </geometry>
-        <material name="black">
-            <color rgba="0 0 0 1"/>
-        </material>
-    </visual>
-    <collision>
-        <origin xyz="0 0 0" rpy="0 0 0 "/>
-        <geometry>
-            <cylinder radius="${wheel_radius}" length="${wheel_length}"/>
-        </geometry>
-    </collision>
-    <inertial>
-        <mass value="${wheel_mass}"/>
-        <inertia
-            ixx="0.0001"
-            iyy="0.0001"
-            ixy="0"
-            ixz="0"
-            iyz="0"
-            izz="0.0001"/>
-        <origin xyz="0 0 0" rpy="0 0 0 "/>
-    </inertial>
-</link>
-<link name="laser_link">
-    <visual>
-        <geometry>
-            <cylinder length="0.06" radius="0.04"/>
-        </geometry>
-        <material name="white">
-            <color rgba="1 1 1 1"/>
-        </material>
-    </visual>
-</link>
-<joint name="laser_joint" type="fixed">
-    <parent link="base_link"/>
-    <child link="laser_link"/>
-    <origin xyz="0 0.0 0.06"/>
-</joint>
+        <origin xyz="-0.1 0.09 -0.03" rpy="1.5707 0 0"/>
+        <parent link="base_link"/>
+        <child link="left_wheel_link2"/>
+        <axis xyz="0 0 -1"/>
+    </joint>
+    <link name="right_wheel_link2">
+        <visual>
+            <geometry>
+                <cylinder radius="${wheel_radius}" length="${wheel_length}"/>
+            </geometry>
+            <material name="black">
+                <color rgba="0 0 0 1"/>
+            </material>
+        </visual>
+        <collision>
+            <origin xyz="0 0 0" rpy="0 0 0 "/>
+            <geometry>
+                <cylinder radius="${wheel_radius}" length="${wheel_length}"/>
+            </geometry>
+        </collision>
+        <inertial>
+            <mass value="${wheel_mass}"/>
+            <inertia
+                ixx="0.0001"
+                iyy="0.0001"
+                ixy="0"
+                ixz="0"
+                iyz="0"
+                izz="0.0001"/>
+            <origin xyz="0 0 0" rpy="0 0 0 "/>
+        </inertial>
+    </link>
+    <joint name="right_wheel_joint2" type="continuous">
+        <origin xyz="-0.1 -0.09 -0.03" rpy="1.5707 0 0"/>
+        <parent link="base_link"/>
+        <child link="right_wheel_link2"/>
+        <axis xyz="0 0 -1"/>
+    </joint>
+    <link name="laser_link">
+        <visual>
+            <geometry>
+                <cylinder length="0.06" radius="0.04"/>
+            </geometry>
+            <material name="white">
+                <color rgba="1 1 1 1"/>
+            </material>
+        </visual>
+    </link>
+    <joint name="laser_joint" type="fixed">
+        <parent link="base_link"/>
+        <child link="laser_link"/>
+        <origin xyz="0 0.0 0.06"/>
+    </joint>
     <!-- <joint name="caster_joint" type="continuous">
         <origin xyz="0 0 0" rpy="-0.10 0 -0.03"/>

File: my_robot_description/urdf/xacro/gazebo/my_robot_with_laser_gazebo.xacro (robot description, xacro)
@@ -1,17 +1,42 @@
 <?xml version="1.0"?>
-<robot name="arm" xmlns:xacro="http://www.ros.org/wiki/xacro">
-    <xacro:include filename="$(find my_robot_description)/urdf/xacro/gazebo/my_robot_base_gazebo.xacro" />
-    <xacro:include filename="$(find my_robot_description)/urdf/xacro/sensors/lidar_gazebo.xacro" />
-    <xacro:property name="lidar_offset_x" value="0" />
-    <xacro:property name="lidar_offset_y" value="0" />
-    <xacro:property name="lidar_offset_z" value="0.105" />
-    <my_robot_base/>
-    <!-- lidar -->
-    <joint name="lidar_joint" type="fixed">
-        <origin xyz="${lidar_offset_x} ${lidar_offset_y} ${lidar_offset_z}" rpy="0 0 0" />
-        <parent link="base_link"/>
-        <child link="laser_link"/>
-    </joint>
-    <xacro:rplidar prefix="laser"/>
-    <my_robot_base_gazebo/>
+<robot name="my_laser" xmlns:xacro="http://www.ros.org/wiki/xacro">
+ <gazebo reference="laser_link">
+     <sensor type="ray" name="rplidar_sensor">
+      <pose>0 0 0 0 0 0</pose>
+      <visualize>true</visualize>
+      <update_rate>40</update_rate>
+      <ray>
+        <scan>
+          <horizontal>
+            <samples>720</samples>
+            <resolution>0.5</resolution>
+            <min_angle>0.0</min_angle>
+            <max_angle>6.28319</max_angle>
+          </horizontal>
+        </scan>
+        <range>
+          <min>0.120</min>
+          <max>12.0</max>
+          <resolution>0.015</resolution>
+        </range>
+        <noise>
+          <type>gaussian</type>
+          <!-- Noise parameters based on published spec for Hokuyo laser
+               achieving "+-30mm" accuracy at range < 10m.  A mean of 0.0m and
+               stddev of 0.01m will put 99.7% of samples within 0.03m of the true
+               reading. -->
+          <mean>0.0</mean>
+          <stddev>0.01</stddev>
+        </noise>
+      </ray>
+      <plugin name="gazebo_ros_ray_sensor" filename="libgazebo_ros_ray_sensor.so">
+        <ros>
+                  <!-- 重映射输出的话题名称 -->
+                  <remapping>~/out:=scan</remapping>
+          </ros>
+          <output_type>sensor_msgs/LaserScan</output_type>
+          <frameName>laser_link</frameName>
+      </plugin>
+    </sensor>
+  </gazebo>
 </robot>
