Commit message: 导航功能开通

File: my_robot_description/urdf/xacro/gazebo/my_robot_base_gazebo.xacro (robot description, xacro)
@@ -3,181 +3,117 @@
     <xacro:include filename="$(find my_robot_description)/urdf/xacro/gazebo/my_robot_control.xacro" />
     <xacro:include filename="$(find my_robot_description)/urdf/xacro/gazebo/my_robot_with_laser_gazebo.xacro" />
-    <xacro:property name="base_mass" value="0.1"/>
-    <xacro:property name="base_radius" value="0.20"/>
-    <xacro:property name="base_length" value="0.16"/>
-    <xacro:property name="wheel_mass" value="0.1"/>
-    <xacro:property name="wheel_radius" value="0.025"/>
-    <xacro:property name="wheel_length" value="0.02"/>
-    <xacro:property name="wheel_joint_y" value="0.19"/>
-    <xacro:property name="caster_radius" value="0.025"/>
     <link name="base_footprint">
-        <origin rpy="0 0 0 " xyz="0 0 0"/>
+      <origin rpy="0 0 0" xyz="0 0 0 "/>
     </link>
-    <link name="base_link">
-        <visual>
-            <geometry>
-                <box size="0.25 0.16 0.05"/>
-            </geometry>
-            <origin rpy="0 0 0 " xyz="0 0 0 "/>
-            <!-- <material name="blue">
-                <color rgba="0 0 0.8 1"/>
-            </material> -->
-        </visual>
-        <collision>
-            <origin rpy="0 0 0 " xyz="0 0 0 "/>
-            <geometry>
-                <box size="0.25 0.16 0.05"/>
-            </geometry>
-        </collision>
-        <inertial>
-            <origin rpy="0 0 0 " xyz="0 0 0 "/>
-            <mass value="${base_mass}"/>
-            <inertia
-                ixx="0.0001"
-                iyy="0.0001"
-                ixy="0"
-                ixz="0"
-                iyz="0"
-                izz="0.0001"/>
-        </inertial>
-    </link>
-    <joint name="base_joint" type="fixed">
-        <parent link="base_footprint"/>
-        <child link="base_link"/>
-        <origin rpy="0 0 0 " xyz="7 4 0.025"/>
-    </joint>
-    <link name="left_wheel_link1">
-        <visual>
-            <geometry>
-                <cylinder radius="${wheel_radius}" length="${wheel_length}"/>
-            </geometry>
-            <material name="black">
-                <color rgba="0 0 0 1"/>
-            </material>
-        </visual>
-        <collision>
-            <origin xyz="0 0 0" rpy="0 0 0 "/>
-            <geometry>
-                <cylinder radius="${wheel_radius}" length="${wheel_length}"/>
-            </geometry>
-        </collision>
-        <inertial>
-           <mass value="${wheel_mass}"/>
-            <inertia
-                ixx="0.0001"
-                iyy="0.0001"
-                ixy="0"
-                ixz="0"
-                iyz="0"
-                izz="0.0001"/>
-            <origin xyz="0 0 0" rpy="0 0 0 "/>
-        </inertial>
-    </link>
-    <joint name="left_wheel_joint1" type="continuous">
-        <origin xyz="0.1 0.09 -0.03" rpy="1.5707 0 0"/>
-        <parent link="base_link"/>
-        <child link="left_wheel_link1"/>
-        <axis xyz="0 0 -1"/>
-    </joint>
-    <link name="right_wheel_link1">
-        <visual>
-            <geometry>
-                <cylinder radius="${wheel_radius}" length="${wheel_length}"/>
-            </geometry>
-            <material name="black">
-                <color rgba="0 0 0 1"/>
-            </material>
-        </visual>
-        <collision>
-            <origin xyz="0 0 0" rpy="0 0 0 "/>
-            <geometry>
-                <cylinder radius="${wheel_radius}" length="${wheel_length}"/>
-            </geometry>
-        </collision>
-        <inertial>
-            <mass value="${wheel_mass}"/>
-            <inertia
-                ixx="0.0001"
-                iyy="0.0001"
-                ixy="0"
-                ixz="0"
-                iyz="0"
-                izz="0.0001"/>
-            <origin xyz="0 0 0" rpy="0 0 0 "/>
-        </inertial>
-    </link>
-    <joint name="right_wheel_joint1" type="continuous">
-        <origin xyz="0.1 -0.09 -0.03" rpy="1.5707 0 0"/>
-        <parent link="base_link"/>
-        <child link="right_wheel_link1"/>
-        <axis xyz="0 0 -1"/>
-    </joint>
-    <link name="left_wheel_link2">
-        <visual>
-            <geometry>
-                <cylinder radius="${wheel_radius}" length="${wheel_length}"/>
-            </geometry>
-            <material name="black">
-                <color rgba="0 0 0 1"/>
-            </material>
-        </visual>
-        <collision>
-            <origin xyz="0 0 0" rpy="0 0 0 "/>
-            <geometry>
-                <cylinder radius="${wheel_radius}" length="${wheel_length}"/>
-            </geometry>
-        </collision>
-        <inertial>
-            <mass value="${wheel_mass}"/>
-            <inertia
-                ixx="0.0001"
-                iyy="0.0001"
-                ixy="0"
-                ixz="0"
-                iyz="0"
-                izz="0.0001"/>
-            <origin xyz="0 0 0" rpy="0 0 0 "/>
-        </inertial>
-    </link>
-    <joint name="left_wheel_joint2" type="continuous">
-        <origin xyz="-0.1 0.09 -0.03" rpy="1.5707 0 0"/>
-        <parent link="base_link"/>
-        <child link="left_wheel_link2"/>
-        <axis xyz="0 0 -1"/>
-    </joint>
-    <link name="right_wheel_link2">
-        <visual>
-            <geometry>
-                <cylinder radius="${wheel_radius}" length="${wheel_length}"/>
-            </geometry>
-            <material name="black">
-                <color rgba="0 0 0 1"/>
-            </material>
-        </visual>
-        <collision>
-            <origin xyz="0 0 0" rpy="0 0 0 "/>
-            <geometry>
-                <cylinder radius="${wheel_radius}" length="${wheel_length}"/>
-            </geometry>
-        </collision>
-        <inertial>
-            <mass value="${wheel_mass}"/>
-            <inertia
-                ixx="0.0001"
-                iyy="0.0001"
-                ixy="0"
-                ixz="0"
-                iyz="0"
-                izz="0.0001"/>
-            <origin xyz="0 0 0" rpy="0 0 0 "/>
-        </inertial>
-    </link>
-    <joint name="right_wheel_joint2" type="continuous">
-        <origin xyz="-0.1 -0.09 -0.03" rpy="1.5707 0 0"/>
-        <parent link="base_link"/>
-        <child link="right_wheel_link2"/>
-        <axis xyz="0 0 -1"/>
-    </joint>
-    <link name="laser_link">
+  <joint name="base_joint" type="fixed">
+    <parent link="base_footprint"/>
+    <child link="base_link"/>
+    <origin rpy="0 0 0" xyz="0 0 0"/>
+  </joint>
+  <link name="base_link">
+    <inertial>
+     <origin xyz="0 0 0" rpy="0 0 0"/>
+     <mass value="0.1"/>
+     <inertia ixx="0.0001"  ixy="0"  ixz="0" iyy="0.0001" iyz="0" izz="0.001" />
+    </inertial>
+    <visual>
+      <geometry>
+        <box size="0.25 0.16 0.05"/>
+      </geometry>
+      <origin rpy="0 0 0" xyz="0 0 0"/>
+      <material name="blue">
+          <color rgba="0 0 0.8 1"/>
+      </material>
+    </visual>
+   <collision>
+     <origin xyz="0 0 0" rpy="0 0 0"/>
+     <geometry>
+       <box size="0.25 0.16 0.05"/>
+     </geometry>
+   </collision>
+  </link>
+  <link name="right_wheel_link">
+    <inertial>
+     <origin xyz="0 0 0" rpy="0 0 0"/>
+     <mass value="0.1"/>
+     <inertia ixx="0.0001"  ixy="0"  ixz="0" iyy="0.0001" iyz="0" izz="0.0001" />
+    </inertial>
+    <visual>
+      <geometry>
+        <cylinder length="0.02" radius="0.025"/>
+      </geometry>
+      <material name="black">
+        <color rgba="0 0 0 1"/>
+      </material>
+    </visual>
+    <collision>
+     <origin xyz="0 0 0" rpy="0 0 0"/>
+     <geometry>
+       <cylinder length="0.02" radius="0.025"/>
+     </geometry>
+    </collision>
+  </link>
+  <joint name="right_wheel_joint" type="continuous">
+    <axis xyz="0 0 -1"/>
+    <parent link="base_link"/>
+    <child link="right_wheel_link"/>
+    <origin rpy="1.5707 0 0" xyz=" 0.1 -0.09 -0.03"/>
+    <!-- <dynamics damping="0.1" friction="0.1"/> 添加摩擦和阻尼 -->
+  </joint>
+  <link name="left_wheel_link">
+    <inertial>
+     <origin xyz="0 0 0" rpy="0 0 0"/>
+     <mass value="0.1"/>
+     <inertia ixx="0.0001"  ixy="0"  ixz="0" iyy="0.0001" iyz="0" izz="0.0001" />
+    </inertial>
+    <visual>
+      <geometry>
+        <cylinder length="0.02" radius="0.025"/>
+      </geometry>
+      <material name="black">
+        <color rgba="0 0 0 1"/>
+      </material>
+    </visual>
+    <collision>
+     <origin xyz="0 0 0" rpy="0 0 0"/>
+     <geometry>
+       <cylinder length="0.02" radius="0.025"/>
+     </geometry>
+    </collision>
+  </link>
+  <joint name="left_wheel_joint" type="continuous">
+    <axis xyz="0 0 -1"/>
+    <parent link="base_link"/>
+    <child link="left_wheel_link"/>
+    <origin rpy="1.5707 0 0" xyz="0.1 0.09 -0.03"/>
+  </joint>
+  <link name="ball_wheel_link">
+    <inertial>
+     <origin xyz="0 0 0" rpy="0 0 0"/>
+     <mass value="0.1"/>
+     <inertia ixx="0"  ixy="0"  ixz="0" iyy="0" iyz="0" izz="0" />
+    </inertial>
+    <visual>
+      <geometry>
+        <sphere radius="0.025"/>
+      </geometry>
+      <material name="black">
+        <color rgba="0 0 0 1"/>
+      </material>
+    </visual>
+    <collision>
+     <origin xyz="0 0 0" rpy="0 0 0"/>
+     <geometry>
+       <sphere radius="0.025"/>
+     </geometry>
+    </collision>
+  </link>
+  <joint name="ball_wheel_joint" type="fixed">
+    <axis xyz="0 0 1"/>
+    <parent link="base_link"/>
+    <child link="ball_wheel_link"/>
+    <origin rpy="0 0 0" xyz="-0.10 0 -0.03"/>
+  </joint>
+  <link name="laser_link">
         <visual>
             <geometry>
@@ -194,36 +130,3 @@
         <origin xyz="0 0.0 0.06"/>
     </joint>
-    <!-- <joint name="caster_joint" type="continuous">
-        <origin xyz="0 0 0" rpy="-0.10 0 -0.03"/>
-        <parent link="base_link"/>
-        <child link="caster_link"/>
-        <axis xyz="0 0 1"/>
-    </joint>
-    <link name="caster_link">
-        <visual>
-            <geometry>
-                <sphere radius="${caster_radius}"/>
-            </geometry>
-            <material name="black">
-                <color rgba="0 0 0 1"/>
-            </material>
-        </visual>
-        <collision>
-            <origin xyz="0 0 0" rpy="0 0 0"/>
-            <geometry>
-                <sphere radius="${caster_radius}"/>
-            </geometry>
-        </collision>
-        <inertial>
-            <mass value="${wheel_mass}"/>
-            <origin xyz="0 0 0" rpy="0 0 0"/>
-            <inertia
-                ixx="0"
-                iyy="0"
-                ixy="0"
-                ixz="0"
-                iyz="0"
-                izz="0"/>
-        </inertial>
-    </link> -->
 </robot>

File: my_robot_description/urdf/xacro/gazebo/my_robot_control.xacro (robot description, xacro)
@@ -1,24 +1,27 @@
 <?xml version="1.0"?>
-<robot name="my_control" xmlns:xacro="http://www.ros.org/wiki/xacro">
+<robot name="my_robot" xmlns:xacro="http://www.ros.org/wiki/xacro">
 <gazebo>
-  <plugin name="differential_drive_controller" filename="libgazebo_ros_diff_drive.so">
-    <updateRate>100</updateRate>
-    <left_joint>left_wheel_joint1</left_joint>
-    <right_joint>right_wheel_joint1</right_joint>
+    <plugin name="mybot_controller" filename="libgazebo_ros_diff_drive.so">
+       <ros>
+            <remapping>odom:=odom</remapping>
+        </ros>
+    <commandTopic>cmd_vel</commandTopic>
+    <publish_odom>true</publish_odom>
+    <publish_odom_tf>true</publish_odom_tf>
+    <publish_wheel_tf>true</publish_wheel_tf>
+    <odometry_frame>odom</odometry_frame>
+    <robot_base_frame>base_footprint</robot_base_frame>
+    <publishTf>true</publishTf>
+    <publishWheelJointState>true</publishWheelJointState>
+    <legacyMode>false</legacyMode>
+    <updateRate>30</updateRate>
+    <left_joint>left_wheel_joint</left_joint>
+    <right_joint>right_wheel_joint</right_joint>
     <wheel_separation>0.180</wheel_separation>
     <wheel_diameter>0.05</wheel_diameter>
     <wheelAcceleration>10</wheelAcceleration>
     <wheelTorque>100</wheelTorque>
-    <commandTopic>cmd_vel</commandTopic>
-    <odometryTopic>odom</odometryTopic>
-    <odometryFrame>odom</odometryFrame>
-    <robotBaseFrame>base_footprint</robotBaseFrame>
-    <odometrySource>1</odometrySource>
-    <publishWheelTF>false</publishWheelTF>
-    <publishTF>true</publishTF>
-    <publishOdom>true</publishOdom>
-    <publishWheelJointState>true</publishWheelJointState>
-    <legacyMode>false</legacyMode>
-  </plugin>
-</gazebo>
+    <rosDebugLevel>na</rosDebugLevel>
+    </plugin>
+  </gazebo>
 </robot>

File: my_robot_description/urdf/xacro/gazebo/my_robot_with_laser_gazebo.xacro (robot description, xacro)
@@ -1,8 +1,34 @@
 <?xml version="1.0"?>
-<robot name="my_laser" xmlns:xacro="http://www.ros.org/wiki/xacro">
+<robot name="my_robot" xmlns:xacro="http://www.ros.org/wiki/xacro">
+  <gazebo reference="left_wheel_link">
+    <mu1>1.0</mu1>
+    <mu2>1.0</mu2>
+    <kd>10.0</kd>
+    <minDepth>0.001</minDepth>
+    <maxVel>1.0</maxVel>
+    <fdir1>1 0 0</fdir1>
+    <material>Gazebo/DarkGrey</material>
+  </gazebo>
+  <gazebo reference="right_wheel_link">
+    <mu1>1.0</mu1>
+    <mu2>1.0</mu2>
+    <kd>10.0</kd>
+    <minDepth>0.001</minDepth>
+    <maxVel>1.0</maxVel>
+    <fdir1>1 0 0</fdir1>
+    <material>Gazebo/FlatBlack</material>
+  </gazebo>
+  <gazebo reference="ball_wheel_link">
+    <mu1>0.1</mu1>
+    <mu2>0.1</mu2>
+    <kd>100.0</kd>
+    <minDepth>0.001</minDepth>
+    <maxVel>1.0</maxVel>
+    <material>Gazebo/FlatBlack</material>
+  </gazebo>
  <gazebo reference="laser_link">
      <sensor type="ray" name="rplidar_sensor">
       <pose>0 0 0 0 0 0</pose>
-      <visualize>true</visualize>
+      <visualize>false</visualize>
       <update_rate>40</update_rate>
       <ray>
@@ -30,5 +56,5 @@
         </noise>
       </ray>
-      <plugin name="gazebo_ros_ray_sensor" filename="libgazebo_ros_ray_sensor.so">
+      <plugin name="gazebo_ros_rplidar_controller" filename="libgazebo_ros_ray_sensor.so">
         <ros>
                   <!-- 重映射输出的话题名称 -->
